File: lose_power_unit/lose_power_unit.kicad_pcb (KiCad board)
At the start: 2 copper layers, 14.5 x 9 mm, 15 parts, among them J1 Conn_01x01_Pin, J2 Conn_01x01_Pin, J3 Conn_01x01_Pin, J4 Conn_01x01_Pin, U1 LM317_SOT-223

Commit message: made the production files
Parts:
- C1: footprint Capacitor_SMD:C_0603_1608Metric -> Capacitor_SMD:C_0402_1005Metric
- turned R1 to 90 degrees
- turned R2 to 90 degrees
Connections:
- R1 pad 1: Net-(D5-A) -> VCC
- R1 pad 2: VCC -> Net-(D5-A)
- R2 pad 1: Net-(R2-Pad1) -> Net-(U1-VO)
- R2 pad 2: Net-(U1-VO) -> Net-(R2-Pad2)
- RV1 pad 3: Net-(R2-Pad1) -> Net-(R2-Pad2)
Routing:
- net Net-(J3-Pin_1): track 0.00 -> 15.5 mm, vias 0 -> 2
- net VCC: track 0.00 -> 15.1 mm
- net Net-(U1-VO): track 0.00 -> 9.36 mm
- net Net-(R2-Pad2): track 0.00 -> 8.69 mm, vias 0 -> 2
- net Net-(D5-A): track 0.00 -> 5.62 mm, vias 0 -> 1
- net AC1: track 0.00 -> 4.53 mm, vias 0 -> 1
- net AC2: track 0.00 -> 3.87 mm, vias 0 -> 1
- net GND: track 0.00 -> 1.97 mm, vias 0 -> 1
- added copper zone on B.Cu, net GND
- added copper zone on F.Cu, net GND
Other:
- board text added: "+"
- board text added: "-"
- board text added: "DCC"
- board text added: "~"
